File: board/kicad/kicad.kicad_pcb (KiCad board)
At the start: 2 copper layers, 220.5 x 101.8 mm, 26 parts

Commit message: feat: PCB routed
Connections:
- D5 pad 2: (no net) -> P28
Routing:
- net P7: track 0.00 -> 262.4 mm, vias 0 -> 2
- net P2: track 0.00 -> 252.9 mm, vias 0 -> 2
- net P0: track 0.00 -> 238.9 mm, vias 0 -> 2
- net P1: track 0.00 -> 233.7 mm, vias 0 -> 4
- net mirror_home_default: track 0.00 -> 100.0 mm, vias 0 -> 1
- net P28: track 0.00 -> 89.0 mm
- net mirror_outer_default: track 0.00 -> 78.3 mm, vias 0 -> 1
- net P4: track 0.00 -> 69.1 mm
- net P6: track 0.00 -> 68.5 mm
- net P29: track 0.00 -> 64.9 mm
- net P5: track 0.00 -> 63.9 mm
- net pinky_top: track 0.00 -> 53.0 mm, vias 0 -> 1
- net pinky_home: track 0.00 -> 51.0 mm, vias 0 -> 1
- net mirror_pinky_top: track 0.00 -> 42.4 mm, vias 0 -> 1
- net mirror_pinky_home: track 0.00 -> 37.0 mm, vias 0 -> 1
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- added copper zone on B.Cu, net GND
- added copper zone on F.Cu, net GND
